File: MasterModule/PCB/Bus/BusModule/BusModule.kicad_pcb (KiCad board)
At the start: 2 copper layers, 65 x 42.5 mm, 6 parts

Commit message: [BUS] Add coper fields
Parts:
- added CAN_0: Conn_01x02, Connector_JST:JST_XH_B2B-XH-A_1x02_P2.50mm_Vertical, F.Cu at (109.7, 120.7)
- added CAN_1: Conn_01x02, Connector_JST:JST_XH_B2B-XH-A_1x02_P2.50mm_Vertical, F.Cu at (68.6, 123.2)
- added POW_0: Conn_01x02, TerminalBlock:TerminalBlock_MaiXu_MX126-5.0-02P_1x02_P5.00mm, F.Cu at (109.2, 103.0)
- added POW_1: Conn_01x02, TerminalBlock:TerminalBlock_MaiXu_MX126-5.0-02P_1x02_P5.00mm, F.Cu at (69.1, 107.5)
- added Pump_0: Conn_01x04, Connector_JST:JST_XH_B4B-XH-A_1x04_P2.50mm_Vertical, F.Cu at (92.6, 125.7)
- added Pump_1: Conn_01x04, Connector_JST:JST_XH_B4B-XH-A_1x04_P2.50mm_Vertical, F.Cu at (84.6, 125.7)
Routing:
- net +12V: track 96.4 -> 192.8 mm
- net GND: track 50.9 -> 101.7 mm
- net /CAN_L: track 44.2 -> 88.5 mm
- net /CAN_H: track 43.2 -> 86.5 mm
- net (no net): vias 4 -> 8
Other:
- board size 65 x 42.5 mm -> 92.5 x 110 mm

Commit message: [PCB][BUS] Fix power connections plates (v 1.2)
Parts:
- removed the CAN_0 at (109.7, 120.7)
- removed the CAN_1 at (68.6, 123.2)
- removed the POW_0 at (109.2, 103.0)
- removed the POW_1 at (69.1, 107.5)
- removed the Pump_0 at (92.6, 125.7)
- removed the Pump_1 at (84.6, 125.7)
Routing:
- net +12V: track 192.8 -> 96.4 mm
- net GND: track 101.7 -> 50.9 mm
- net /CAN_L: track 88.5 -> 44.2 mm
- net /CAN_H: track 86.5 -> 43.2 mm
- net (no net): vias 8 -> 4
Other:
- board size 92.5 x 110 mm -> 92.5 x 42.5 mm
- board text added: "Bus v1.2"
- board text removed: "Bus v1.1"
