File: MasterModule/PCB/Bus/BusModule/BusModule.kicad_pcb (KiCad board)
At the start: 2 copper layers, 92.5 x 42.5 mm, 6 parts

Commit message: [Bus][PCB] Create manufacturing files for 2 PCB v1.2
Parts:
- added CAN_0: Conn_01x02, Connector_JST:JST_XH_B2B-XH-A_1x02_P2.50mm_Vertical, F.Cu at (109.2, 116.0)
- added CAN_1: Conn_01x02, Connector_JST:JST_XH_B2B-XH-A_1x02_P2.50mm_Vertical, F.Cu at (68.1, 118.5)
- added POW_0: Conn_01x02, TerminalBlock:TerminalBlock_MaiXu_MX126-5.0-02P_1x02_P5.00mm, F.Cu at (108.7, 98.2)
- added POW_1: Conn_01x02, TerminalBlock:TerminalBlock_MaiXu_MX126-5.0-02P_1x02_P5.00mm, F.Cu at (68.6, 102.8)
- added Pump_0: Conn_01x04, Connector_JST:JST_XH_B4B-XH-A_1x04_P2.50mm_Vertical, F.Cu at (92.1, 121.0)
- added Pump_1: Conn_01x04, Connector_JST:JST_XH_B4B-XH-A_1x04_P2.50mm_Vertical, F.Cu at (84.1, 121.0)
- moved CAN_0 1.12 mm to (109.2, 72.2)
- moved CAN_1 1.12 mm to (68.1, 74.7)
- moved POW_0 1.12 mm to (108.7, 54.5)
- moved POW_1 1.12 mm to (68.6, 59.0)
- moved Pump_0 1.12 mm to (92.1, 77.2)
- moved Pump_1 1.12 mm to (84.1, 77.2)
Routing:
- net +12V: track 96.4 -> 192.8 mm
- net GND: track 50.9 -> 101.7 mm
- net /CAN_L: track 44.2 -> 88.5 mm
- net /CAN_H: track 43.2 -> 86.5 mm
- net (no net): vias 4 -> 8
Other:
- board size 92.5 x 42.5 mm -> 65 x 86.2 mm
