File: MasterModule/PCB/Bus/BusModule/_restore_backup_2026-05-27T22-22-10-652/BusModule.kicad_pcb (KiCad board)
At the start: 2 copper layers, 65 x 42.5 mm, 6 parts

Commit message: [PCB][Bus] Add GND and 12V poligon (Bus v1.1)
Routing:
- removed copper zone on B.Cu, net +12V
- removed copper zone on B.Cu, net GND
Other:
- board text added: "Bus v1.0"
- board text removed: "Bus v1.1"
Changed lines of the file:
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@@
 		(filling no)
 		(pcbplotparams
-			(layerselection 0x00000000_00000000_55555555_55555550)
-			(plot_on_all_layers_selection 0x00000000_00000000_00000000_02000000)
+			(layerselection 0x00000000_00000000_55555555_55555558)
+			(plot_on_all_layers_selection 0x00000000_00000000_00000000_00000000)
 			(disableapertmacros no)
 			(usegerberextensions no)
@@
 			(crossoutdnponfab yes)
 			(subtractmaskfromsilk no)
-			(outputformat 1)
-			(mirror no)
+			(outputformat 4)
+			(mirror yes)
 			(drillshape 0)
 			(scaleselection 1)
@@
 		(layer "Edge.Cuts")
 	)
-	(gr_text "Bus v1.1"
+	(gr_text "Bus v1.0"
 		(at 94 50 0)
 		(layer "B.Cu")
@@
 		)
 	)
-	(gr_text "Bus v1.1"
+	(gr_text "Bus v1.0"
 		(at 79 52 0)
 		(layer "F.SilkS")
@@
 		(net "/CAN_H")
 	)
-	(zone
-		(net "+12V")
-		(layer "B.Cu")
-		(hatch edge 0.5)
-		(priority 1)
-		(connect_pads
-			(clearance 1)
-		)
-		(min_thickness 0.25)
-		(fill yes
-			(thermal_gap 0.5)
-			(thermal_bridge_width 0.5)
-			(island_removal_mode 0)
-		)
-		(polygon
-			(pts
-				(xy 69 54.75) (xy 84.5 70.5) (xy 92.75 70.5) (xy 108.75 55.25)
-			)
-		)
-	)
-	(zone
-		(net "GND")
-		(layer "B.Cu")
-		(hatch edge 0.5)
-		(connect_pads
-			(clearance 1)
-		)
-		(min_thickness 0.25)
-		(fill yes
-			(thermal_gap 0.5)
-			(thermal_bridge_width 0.5)
-			(island_removal_mode 0)
-		)
-		(polygon
-			(pts
-				(xy 57.5 87.5) (xy 57.5 45) (xy 122.5 45) (xy 122.5 87.5)
-			)
-		)
-	)
 	(embedded_fonts no)
