File: MasterModule/PCB/MasterModule/MasterModule/Power_unit.kicad_sch (KiCad schematic)
At the start: 8 parts, among them J1 Input_7V, U1 AMS1117-3.3, U2 AMS1117-5.0

Commit message: [PCB][MasterModule] Fix CAN transmitter to TJA1050 chip (Master v1.1)
Parts:
- C3: footprint Capacitor_SMD:C_0805_2012Metric_Pad1.18x1.45mm_HandSolder -> Capacitor_SMD:C_0603_1608Metric_Pad1.08x0.95mm_HandSolder
Changed lines of the file:
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@@
 			)
 		)
-		(property "Footprint" "Capacitor_SMD:C_0805_2012Metric_Pad1.18x1.45mm_HandSolder"
+		(property "Footprint" "Capacitor_SMD:C_0603_1608Metric_Pad1.08x0.95mm_HandSolder"
 			(at 39.0652 76.2 0)
 			(hide yes)
