File: MasterModule/PCB/MasterModule/MasterModule/UART_galvanic_isolation.kicad_sch (KiCad schematic)
At the start: 0 parts

Commit message: [PCB][MasterModule] Create MasterModule v.1.0
Parts:
- added C4, C5: 10uF, Capacitor_SMD:C_0805_2012Metric_Pad1.18x1.45mm_HandSolder, symbol Device:C
- added J2: UART, Connector_JST:JST_XH_B4B-XH-A_1x04_P2.50mm_Vertical, symbol Connector_Generic:Conn_01x04
- added U3: ADuM1201AR, Package_SO:SOIC-8_3.9x4.9mm_P1.27mm, symbol Isolator:ADuM1201AR
Connections:
- new net: C4.2, J2.1 (Pin_1), U3.5 (GND2)
- new net: J2.2 (Pin_2), U3.6 (VOB)
- new net: J2.3 (Pin_3), U3.7 (VIA)
- new net: C4.1, J2.4 (Pin_4), U3.8 (VDD2)
- new net 3.3V: C5.1, U3.1 (VDD1)
- new net GND: C5.2, U3.4 (GND1)
- new net RX: U3.2 (VOA)
- new net TX: U3.3 (VIB)

Commit message: [PCB][MasterModule] Fix CAN transmitter to TJA1050 chip (Master v1.1)
Parts:
- C4, C5: footprint Capacitor_SMD:C_0805_2012Metric_Pad1.18x1.45mm_HandSolder -> Capacitor_SMD:C_0603_1608Metric_Pad1.08x0.95mm_HandSolder
Changed lines of the file:
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@@
 			)
 		)
-		(property "Footprint" "Capacitor_SMD:C_0805_2012Metric_Pad1.18x1.45mm_HandSolder"
+		(property "Footprint" "Capacitor_SMD:C_0603_1608Metric_Pad1.08x0.95mm_HandSolder"
 			(at 87.3252 88.9 0)
 			(hide yes)
@@
 			)
 		)
-		(property "Footprint" "Capacitor_SMD:C_0805_2012Metric_Pad1.18x1.45mm_HandSolder"
+		(property "Footprint" "Capacitor_SMD:C_0603_1608Metric_Pad1.08x0.95mm_HandSolder"
 			(at 143.2052 88.9 0)
 			(hide yes)
